File: schematics/src/ioboard/ioboard.brd (EAGLE design)
At the start: 80 x 99.1 mm, 31 parts, among them IC1 MCP23S17SP, SW1 EC12E_SW

Commit message: Fixed schematics & descriptions
Parts:
- removed JP1, JP2: (no value), pinhead:2X08
- removed RN3, RN4: (no value), resistor-sil:SIL9
- added IC2: MAX7219CNG, maxim:DIL24-3
Connections:
- new net VCC: IC2.19
- net GND: now also IC2.4, IC2.9; no longer RN3.2, RN4.1
- net N$1: no longer RN3.1
- net N$10: no longer RN4.3
- net N$11: no longer RN4.4
- net N$12: no longer RN4.5
- net N$13: no longer RN4.6
- net N$14: no longer RN4.7
- net N$15: no longer RN4.8
- net N$16: no longer RN4.9
- net N$17: no longer JP1.2
- net N$18: no longer JP1.4
- net N$19: no longer JP1.6
- net N$2: no longer RN3.3
- net N$20: no longer JP1.8
- net N$21: no longer JP1.10
- net N$22: no longer JP1.12
- net N$23: no longer JP1.14
- net N$24: no longer JP1.16
- net N$25: no longer JP1.1
- net N$26: no longer JP1.3
- net N$27: no longer JP1.5
- net N$28: no longer JP1.7
- net N$29: no longer JP1.9
- net N$3: no longer RN3.4
- net N$30: no longer JP1.11
- net N$31: no longer JP1.13
- net N$32: no longer JP1.15
- net N$33: no longer JP2.2
- net N$34: no longer JP2.4
- net N$35: no longer JP2.6
- net N$36: no longer JP2.8
- net N$37: no longer JP2.10
- net N$38: no longer JP2.12
- net N$39: no longer JP2.14
- net N$4: no longer RN3.5
- net N$40: no longer JP2.16
- net N$41: no longer JP2.1
- net N$42: no longer JP2.3
- net N$43: no longer JP2.5
- net N$44: no longer JP2.7
- net N$45: no longer JP2.9
- net N$46: no longer JP2.11
- net N$47: no longer JP2.13
- net N$48: no longer JP2.15
- net N$5: no longer RN3.6
- net N$6: no longer RN3.7
- net N$7: no longer RN3.8
- net N$8: no longer RN3.9
- net N$9: no longer RN4.2
Routing:
- net N$47: track 35.7 -> 2.06 mm
- net N$48: track 21.2 -> 5.28 mm
- net N$46: track 61.5 -> 58.3 mm
- net N$45: track 92.0 -> 88.8 mm
- net N$2: track 14.0 -> 10.8 mm
- net N$1: track 7.62 -> 5.08 mm
- net N$40: track 23.5 -> 21.7 mm
- net N$39: track 37.8 -> 36.0 mm
- net N$38: track 64.6 -> 62.8 mm
